File: m5atom_power_adc/GroveUnit.kicad_sch (KiCad schematic)
At the start: 9 parts, among them J501 GROVE-CONNECTOR, Q501 AO3401A, Q502 MMBT2222A

Commit message: feat: PCBレイアウト完成・ドキュメントにサブシート構成を反映
- m5atom_power_adc: PCBレイアウト完成（80×82.5mm、131部品、ルーティング完了）
- GroveUnit/RelayControl サブシート更新
- CONTEXT.md/README.md: m5atom_power_adc のファイル構成にサブシート3枚・Library.pretty を追記

Co-Authored-By: Claude Sonnet 4.6 <noreply@anthropic.com>
Connections:
- net GND2 renamed GND1
Changed lines of the file:
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@@
 	)
 	(symbol
-		(lib_id "power:GND2")
-		(at 132.08 121.92 0)
+		(lib_id "power:GND1")
+		(at 133.35 91.44 0)
 		(unit 1)
 		(exclude_from_sim no)
@@
 		(fields_autoplaced yes)
 		(property "Reference" "#PWR0502"
-			(at 132.08 128.27 0)
-			(effects
-				(font
-					(size 1.27 1.27)
-				)
-				(hide yes)
-			)
-		)
-		(property "Value" "GND2"
-			(at 132.08 127 0)
+			(at 133.35 97.79 0)
+			(effects
+				(font
+					(size 1.27 1.27)
+				)
+				(hide yes)
+			)
+		)
+		(property "Value" "GND1"
+			(at 133.35 96.52 0)
 			(effects
 				(font
@@
 		)
 		(property "Footprint" ""
-			(at 132.08 121.92 0)
+			(at 133.35 91.44 0)
 			(effects
 				(font
@@
 		)
 		(property "Datasheet" ""
-			(at 132.08 121.92 0)
-			(effects
-				(font
-					(size 1.27 1.27)
-				)
-				(hide yes)
-			)
-		)
-		(property "Description" "Power symbol creates a global label with name \"GND2\" , ground"
-			(at 132.08 121.92 0)
+			(at 133.35 91.44 0)
+			(effects
+				(font
+					(size 1.27 1.27)
+				)
+				(hide yes)
+			)
+		)
+		(property "Description" "Power symbol creates a global label with name \"GND1\" , ground"
+			(at 133.35 91.44 0)
 			(effects
 				(font
@@
 	)
 	(symbol
+		(lib_id "power:GND1")
+		(at 132.08 121.92 0)
+		(unit 1)
+		(exclude_from_sim no)
+		(in_bom yes)
+		(on_board yes)
+		(dnp no)
+		(fields_autoplaced yes)
+		(property "Reference" "#PWR0504"
+			(at 132.08 128.27 0)
+			(effects
+				(font
+					(size 1.27 1.27)
+				)
+				(hide yes)
+			)
+		)
+		(property "Value" "GND1"
+			(at 132.08 127 0)
+			(effects
+				(font
+					(size 1.27 1.27)
+				)
+			)
+		)
+		(property "Footprint" ""
+			(at 132.08 121.92 0)
+			(effects
+				(font
+					(size 1.27 1.27)
+				)
+				(hide yes)
+			)
+		)
+		(property "Datasheet" ""
+			(at 132.08 121.92 0)
+			(effects
+				(font
+					(size 1.27 1.27)
+				)
+				(hide yes)
+			)
+		)
+		(property "Description" "Power symbol creates a global label with name \"GND1\" , ground"
+			(at 132.08 121.92 0)
+			(effects
+				(font
+					(size 1.27 1.27)
+				)
+				(hide yes)
+			)
+		)
+		(pin "1"
+		)
+		(instances
+			(project "m5atom_power_adc"
+				(path "/d0098cfc-b338-460c-a156-403456706079/051dea6d-d386-40cf-8d3d-92f95e1fe925"
+					(reference "#PWR0504")
+					(unit 1)
+				)
+				(path "/d0098cfc-b338-460c-a156-403456706079/80ef8e19-181b-4673-955c-b259ebecd62e"
+					(reference "#PWR0604")
+					(unit 1)
+				)
+			)
+		)
+	)
+	(symbol
 		(lib_id "Transistor_FET:AO3401A")
 		(at 107.95 86.36 180)
@@
 					(unit 1)
 				)
-			)
-		)
-	)
-	(symbol
-		(lib_id "power:GND2")
-		(at 133.35 91.44 0)
-		(unit 1)
-		(exclude_from_sim no)
-		(in_bom yes)
-		(on_board yes)
-		(dnp no)
-		(fields_autoplaced yes)
-		(property "Reference" "#PWR0503"
-			(at 133.35 97.79 0)
-			(effects
-				(font
-					(size 1.27 1.27)
-				)
-				(hide yes)
-			)
-		)
-		(property "Value" "GND2"
-			(at 133.35 96.52 0)
-			(effects
-				(font
-					(size 1.27 1.27)
-				)
-			)
-		)
-		(property "Footprint" ""
-			(at 133.35 91.44 0)
-			(effects
-				(font
-					(size 1.27 1.27)
-				)
-				(hide yes)
-			)
-		)
-		(property "Datasheet" ""
-			(at 133.35 91.44 0)
-			(effects
-				(font
-					(size 1.27 1.27)
-				)
-				(hide yes)
-			)
-		)
-		(property "Description" "Power symbol creates a global label with name \"GND2\" , ground"
-			(at 133.35 91.44 0)
-			(effects
-				(font
-					(size 1.27 1.27)
-				)
-				(hide yes)
-			)
-		)
-		(pin "1"
-		)
-		(instances
-			(project "m5atom_power_adc"
-				(path "/d0098cfc-b338-460c-a156-403456706079/051dea6d-d386-40cf-8d3d-92f95e1fe925"
-					(reference "#PWR0503")
-					(unit 1)
-				)
-				(path "/d0098cfc-b338-460c-a156-403456706079/80ef8e19-181b-4673-955c-b259ebecd62e"
-					(reference "#PWR0603")
-					(unit 1)
-				)

Commit message: chore: PCBネジ穴追加・シルク整理・ロゴ追加・フットプリント修正
- ネジ穴を追加
- シルク文字・ロゴを整理・追加（k_icon フットプリント）
- HY2.0-4PZZ コネクタフットプリントを追加
- 各サブシートのフットプリント修正
- production/ を .gitignore に追加

Co-Authored-By: Claude Sonnet 4.6 <noreply@anthropic.com>
Parts:
- D501, D502: JLC_Num C502526 -> (none); LCSC (none) -> C502526
- J501: footprint 000_Local:HY2.0-4PWB -> 000_Local:HY2.0-4PZZ; JLC_Num C3029460 -> (none); LCSC (none) -> C7429580
- Q501: JLC_Num C15127 -> (none); LCSC (none) -> C15127
- Q502: JLC_Num C8512 -> (none); LCSC (none) -> C8512
- R501: JLC_Num C2906981 -> (none); LCSC (none) -> C2906981
- R502: JLC_Num C2906862 -> (none); LCSC (none) -> C2906862
- TP501, TP502: now left out of the parts list
Changed lines of the file:
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@@
 		(dnp no)
 		(fields_autoplaced yes)
-		(property "Reference" "#PWR0502"
+		(property "Reference" "#PWR0503"
 			(at 133.35 97.79 0)
 			(effects
@@
 			(project "m5atom_power_adc"
 				(path "/d0098cfc-b338-460c-a156-403456706079/051dea6d-d386-40cf-8d3d-92f95e1fe925"
-					(reference "#PWR0502")
-					(unit 1)
-				)
-				(path "/d0098cfc-b338-460c-a156-403456706079/80ef8e19-181b-4673-955c-b259ebecd62e"
-					(reference "#PWR0602")
+					(reference "#PWR0503")
+					(unit 1)
+				)
+				(path "/d0098cfc-b338-460c-a156-403456706079/80ef8e19-181b-4673-955c-b259ebecd62e"
+					(reference "#PWR0603")
 					(unit 1)
 				)
@@
 			)
 		)
-		(property "Footprint" "000_Local:HY2.0-4PWB"
+		(property "Footprint" "000_Local:HY2.0-4PZZ"
 			(at 132.08 104.14 0)
 			(effects
@@
 			)
 		)
-		(property "JLC_Num" "C3029460"
+		(property "LCSC" "C7429580"
 			(at 132.08 104.14 0)
 			(effects
@@
 			)
 		)
-		(property "JLC_Num" "C2906862"
+		(property "LCSC" "C2906862"
 			(at 129.54 76.2 0)
 			(effects
@@
 		(dnp no)
 		(fields_autoplaced yes)
-		(property "Reference" "#PWR0504"
+		(property "Reference" "#PWR0502"
 			(at 132.08 128.27 0)
 			(effects
@@
 			(project "m5atom_power_adc"
 				(path "/d0098cfc-b338-460c-a156-403456706079/051dea6d-d386-40cf-8d3d-92f95e1fe925"
-					(reference "#PWR0504")
-					(unit 1)
-				)
-				(path "/d0098cfc-b338-460c-a156-403456706079/80ef8e19-181b-4673-955c-b259ebecd62e"
-					(reference "#PWR0604")
+					(reference "#PWR0502")
+					(unit 1)
+				)
+				(path "/d0098cfc-b338-460c-a156-403456706079/80ef8e19-181b-4673-955c-b259ebecd62e"
+					(reference "#PWR0602")
 					(unit 1)
 				)
@@
 			)
 		)
-		(property "JLC_Num" "C15127"
+		(property "LCSC" "C15127"
 			(at 107.95 86.36 0)
 			(effects
@@
 		(unit 1)
 		(exclude_from_sim no)
-		(in_bom yes)
+		(in_bom no)
 		(on_board yes)
 		(dnp no)
@@
 			)
 		)
-		(property "JLC_Num" "C2906981"
+		(property "LCSC" "C2906981"
 			(at 114.3 80.01 0)
 			(effects
@@
 		(unit 1)
 		(exclude_from_sim no)
-		(in_bom yes)
+		(in_bom no)
 		(on_board yes)
 		(dnp no)
@@
 			)
 		)
-		(property "JLC_Num" "C8512"
+		(property "LCSC" "C8512"
 			(at 125.73 83.82 90)
 			(effects
@@
 			)
 		)
-		(property "JLC_Num" "C502526"
+		(property "LCSC" "C502526"
 			(at 120.65 110.49 90)
 			(effects
@@
 			)
 		)
-		(property "JLC_Num" "C502526"
+		(property "LCSC" "C502526"
 			(at 123.19 116.84 90)
 			(effects

Commit message: feat: GroveUnitに電源インジケーターLED追加・PCB配置
回路図：電源インジケーターLED（LED+抵抗）を追加
PCB：LED・抵抗のフットプリント配置・配線
CLAUDE.md：KiCadファイル直接編集禁止ルールを追記

Co-Authored-By: Claude Sonnet 4.6 <noreply@anthropic.com>
Parts:
- added D503: LED, LED_SMD:LED_0603_1608Metric, symbol Device:LED
- added R503: 200, Resistor_SMD:R_0603_1608Metric, symbol Device:R_Small
Connections:
- net GND1: now also R503.2
- net at J501.3, Q501.3 (D), TP501.1: now also D503.2 (A)
- new net: D503.1 (K), R503.1
Changed lines of the file:
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@@
+	)
+	(junction
+		(at 120.65 121.92)
+		(diameter 0)
+		(color 0 0 0 0)
+	)
+	(junction
+		(at 110.49 97.79)
+		(diameter 0)
+		(color 0 0 0 0)
 	)
 	(junction
@@
 	(wire
 		(pts
+			(xy 110.49 121.92) (xy 110.49 114.3)
+		)
+		(stroke
+			(width 0)
+			(type default)
+		)
+	)
+	(wire
+		(pts
 			(xy 120.65 106.68) (xy 120.65 100.33)
 		)
@@
 	(wire
 		(pts
-			(xy 125.73 97.79) (xy 105.41 97.79)
+			(xy 125.73 97.79) (xy 110.49 97.79)
 		)
 		(stroke
@@
 	(wire
 		(pts
+			(xy 120.65 121.92) (xy 110.49 121.92)
+		)
+		(stroke
+			(width 0)
+			(type default)
+		)
+	)
+	(wire
+		(pts
 			(xy 114.3 76.2) (xy 114.3 77.47)
 		)
@@
 		(pts
 			(xy 123.19 121.92) (xy 125.73 121.92)
+		)
+		(stroke
+			(width 0)
+			(type default)
+		)
+	)
+	(wire
+		(pts
+			(xy 110.49 97.79) (xy 105.41 97.79)
+		)
+		(stroke
+			(width 0)
+			(type default)
+		)
+	)
+	(wire
+		(pts
+			(xy 110.49 101.6) (xy 110.49 97.79)
 		)
 		(stroke
@@
 			)
 			(justify right)
+		)
+	)
+	(symbol
+		(lib_id "Device:LED")
+		(at 110.49 105.41 90)
+		(unit 1)
+		(exclude_from_sim no)
+		(in_bom yes)
+		(on_board yes)
+		(dnp no)
+		(property "Reference" "D503"
+			(at 103.632 107.188 90)
+			(effects
+				(font
+					(size 1.27 1.27)
+				)
+				(justify right)
+			)
+		)
+		(property "Value" "LED"
+			(at 112.268 105.41 90)
+			(effects
+				(font
+					(size 1.27 1.27)
+				)
+				(justify right)
+			)
+		)
+		(property "Footprint" "LED_SMD:LED_0603_1608Metric"
+			(at 110.49 105.41 0)
+			(effects
+				(font
+					(size 1.27 1.27)
+				)
+				(hide yes)
+			)
+		)
+		(property "Datasheet" "~"
+			(at 110.49 105.41 0)
+			(effects
+				(font
+					(size 1.27 1.27)
+				)
+				(hide yes)
+			)
+		)
+		(property "Description" "Light emitting diode"
+			(at 110.49 105.41 0)
+			(effects
+				(font
+					(size 1.27 1.27)
+				)
+				(hide yes)
+			)
+		)
+		(property "Sim.Pins" "1=K 2=A"
+			(at 110.49 105.41 0)
+			(effects
+				(font
+					(size 1.27 1.27)
+				)
+				(hide yes)
+			)
+		)
+		(property "LCSC" "C965799"
+			(at 110.49 105.41 90)
+			(effects
+				(font
+					(size 1.27 1.27)
+				)
+				(hide yes)
+			)
+		)
+		(pin "1"
+		)
+		(pin "2"
+		)
+		(instances
+			(project "m5atom_power_adc"
+				(path "/d0098cfc-b338-460c-a156-403456706079/051dea6d-d386-40cf-8d3d-92f95e1fe925"
+					(reference "D503")
+					(unit 1)
+				)
+				(path "/d0098cfc-b338-460c-a156-403456706079/80ef8e19-181b-4673-955c-b259ebecd62e"
+					(reference "D603")
+					(unit 1)
+				)
+			)
 		)
 	)
@@
 	)
 	(symbol
+		(lib_id "Device:R_Small")
+		(at 110.49 111.76 0)
+		(unit 1)
+		(exclude_from_sim no)
+		(in_bom yes)
+		(on_board yes)
+		(dnp no)
+		(property "Reference" "R503"
+			(at 105.156 112.776 0)
+			(effects
+				(font
+					(size 1.016 1.016)
+				)
+				(justify left)
+			)
+		)
+		(property "Value" "200"
+			(at 105.156 115.316 0)
+			(effects
+				(font
+					(size 1.27 1.27)
+				)
+				(justify left)
+			)
+		)
+		(property "Footprint" "Resistor_SMD:R_0603_1608Metric"
+			(at 110.49 111.76 0)
+			(effects
+				(font
+					(size 1.27 1.27)
+				)
+				(hide yes)
+			)
+		)
+		(property "Datasheet" "~"
+			(at 110.49 111.76 0)
+			(effects
+				(font
+					(size 1.27 1.27)
+				)
+				(hide yes)
+			)
+		)
+		(property "Description" "Resistor, small symbol"
+			(at 110.49 111.76 0)
+			(effects
+				(font
+					(size 1.27 1.27)
+				)
+				(hide yes)
+			)
+		)
+		(property "LCSC" "C8218"
+			(at 110.49 111.76 0)
+			(effects
+				(font
+					(size 1.27 1.27)
+				)
+				(hide yes)
+			)
+		)
+		(pin "2"
+		)
+		(pin "1"
+		)
+		(instances
+			(project "m5atom_power_adc"
+				(path "/d0098cfc-b338-460c-a156-403456706079/051dea6d-d386-40cf-8d3d-92f95e1fe925"
+					(reference "R503")
+					(unit 1)
+				)
+				(path "/d0098cfc-b338-460c-a156-403456706079/80ef8e19-181b-4673-955c-b259ebecd62e"
+					(reference "R603")
+					(unit 1)
+				)
+			)
+		)
+	)
+	(symbol
 		(lib_id "power:+5V")
 		(at 114.3 76.2 0)
@@
 		(dnp no)
 		(property "Reference" "D501"
-			(at 111.506 110.49 90)
+			(at 114.046 110.49 90)
 			(effects
 				(font
@@
 		)
 		(property "Value" "SD03"
-			(at 111.506 113.03 90)
-			(effects
-				(font
+			(at 114.046 113.03 90)
+			(effects
+				(font

Commit message: chore: KiCadプロジェクト更新（回路図・PCBレイアウト各種修正）
Co-Authored-By: Claude Sonnet 4.6 <noreply@anthropic.com>
Parts:
- added C501: 47uF, Capacitor_SMD:C_1206_3216Metric, symbol Device:C_Small
- added C502: 100nF, Capacitor_SMD:C_0603_1608Metric, symbol Device:C_Small
- renumbered D503 to D501, D501 to D502, D502 to D503, R503 to R501, R501 to R502, R502 to R503
Connections:
- net +5V: now also C501.1, C502.1
- net GND1: now also C501.2, C502.2

Commit message: chore: Grove LED色変更・リレー抵抗を680Ω 500mWに変更・INA228品番更新
Co-Authored-By: Claude Sonnet 4.6 <noreply@anthropic.com>
Parts:
- D501: LCSC C965799 -> C965804
Changed lines of the file:
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@@
 			)
 		)
-		(property "LCSC" "C965799"
+		(property "LCSC" "C965804"
 			(at 110.49 105.41 90)
 			(effects

Commit message: feat: m5atom_power_adc 回路・PCB を更新
KiCad 上で行った回路設計・PCB レイアウト変更を反映。
変更内容の詳細は KiCad 上で差分を確認すること。

Co-Authored-By: Claude Sonnet 4.6 <noreply@anthropic.com>
Parts:
- R501: value 200 -> 390; LCSC C8218 -> C23151
- R502: LCSC C2906981 -> C25803
- R503: footprint Resistor_SMD:R_0402_1005Metric -> Resistor_SMD:R_0603_1608Metric; LCSC C2906862 -> C25804
Connections:
- net GND1: now also J501.1; no longer J501.4
- net Pin1: now also J501.4; no longer J501.1
- net Pin2: now also J501.3; no longer J501.2
- net at D501.2 (A), Q501.3 (D), TP501.1: now also J501.2; no longer J501.3
Changed lines of the file:
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@@
+	(wire
+		(pts
+			(xy 123.19 102.87) (xy 128.27 102.87)
+		)
+		(stroke
+			(width 0)
+			(type default)
+		)
+	)
+	(wire
+		(pts
+			(xy 120.65 100.33) (xy 128.27 100.33)
+		)
+		(stroke
+			(width 0)
+			(type default)
+		)
+	)
 	(wire
 		(pts
@@
 	(wire
 		(pts
-			(xy 120.65 100.33) (xy 128.27 100.33)
-		)
-		(stroke
-			(width 0)
-			(type default)
-		)
-	)
-	(wire
-		(pts
-			(xy 128.27 105.41) (xy 125.73 105.41)
-		)
-		(stroke
-			(width 0)
-			(type default)
-		)
-	)
-	(wire
-		(pts
 			(xy 132.08 71.12) (xy 132.08 76.2)
 		)
@@
 	(wire
 		(pts
-			(xy 123.19 102.87) (xy 128.27 102.87)
-		)
-		(stroke
-			(width 0)
-			(type default)
-		)
-	)
-	(wire
-		(pts
 			(xy 120.65 121.92) (xy 110.49 121.92)
 		)
@@
 		(pts
 			(xy 105.41 81.28) (xy 105.41 76.2)
+		)
+		(stroke
+			(width 0)
+			(type default)
+		)
+	)
+	(wire
+		(pts
+			(xy 125.73 105.41) (xy 128.27 105.41)
 		)
 		(stroke
@@
 		(lib_id "OPL_Connector:GROVE-CONNECTOR-DIP_4P-2.0_")
 		(at 132.08 104.14 0)
+		(mirror x)
 		(unit 1)
 		(exclude_from_sim no)
@@
 		(on_board yes)
 		(dnp no)
-		(fields_autoplaced yes)
 		(property "Reference" "J501"
+			(at 137.16 105.41 0)
+			(effects
+				(font
+					(size 1.143 1.143)
+				)
+				(justify left)
+			)
+		)
+		(property "Value" "GROVE-CONNECTOR"
 			(at 137.16 102.87 0)
-			(effects
-				(font
-					(size 1.143 1.143)
-				)
-				(justify left)
-			)
-		)
-		(property "Value" "GROVE-CONNECTOR"
-			(at 137.16 105.41 0)
 			(effects
 				(font
@@
 		)
 		(property "SKU" "320110033"
-			(at 132.842 100.33 0)
+			(at 132.842 107.95 0)
 			(effects
 				(font
@@
 			)
 		)
-		(property "Footprint" "Resistor_SMD:R_0402_1005Metric"
+		(property "Footprint" "Resistor_SMD:R_0603_1608Metric"
 			(at 129.54 76.2 0)
 			(effects
@@
 			)
 		)
-		(property "LCSC" "C2906862"
+		(property "LCSC" "C25804"
 			(at 129.54 76.2 0)
 			(effects
@@
 			)
 		)
-		(property "LCSC" "C2906981"
+		(property "LCSC" "C25803"
 			(at 114.3 80.01 0)
 			(effects
@@
 			)
 		)
-		(property "Value" "200"
+		(property "Value" "390"
 			(at 105.156 115.316 0)
 			(effects
@@
 			)
 		)
-		(property "LCSC" "C8218"
+		(property "LCSC" "C23151"
 			(at 110.49 111.76 0)
 			(effects
