File: m5atom_power_adc/VoltageSense.kicad_sch (KiCad schematic)
At the start: 8 parts

Commit message: chore: PCBネジ穴追加・シルク整理・ロゴ追加・フットプリント修正
- ネジ穴を追加
- シルク文字・ロゴを整理・追加（k_icon フットプリント）
- HY2.0-4PZZ コネクタフットプリントを追加
- 各サブシートのフットプリント修正
- production/ を .gitignore に追加

Co-Authored-By: Claude Sonnet 4.6 <noreply@anthropic.com>
Parts:
- C701, C702: JLC_Num C77069 -> (none); LCSC (none) -> C77069
- C703: JLC_Num C464977 -> (none); LCSC (none) -> C464977
- R701: JLC_Num C2989042 -> (none); LCSC (none) -> C2989042
- R702: JLC_Num C326601 -> (none); LCSC (none) -> C326601
- R703, R704: JLC_Num C705627 -> (none); LCSC (none) -> C705627
- TP701: now left out of the parts list
Changed lines of the file:
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@@
 			)
 		)
-		(property "JLC_Num" "C326601"
+		(property "LCSC" "C326601"
 			(at 110.49 95.25 90)
 			(effects
@@
 			)
 		)
-		(property "JLC_Num" "C77069"
+		(property "LCSC" "C77069"
 			(at 129.54 99.06 0)
 			(effects
@@
 		(unit 1)
 		(exclude_from_sim no)
-		(in_bom yes)
+		(in_bom no)
 		(on_board yes)
 		(dnp no)
@@
 			)
 		)
-		(property "JLC_Num" "C2989042"
+		(property "LCSC" "C2989042"
 			(at 105.41 90.17 90)
 			(effects
@@
 			)
 		)
-		(property "JLC_Num" "C705627"
+		(property "LCSC" "C705627"
 			(at 119.38 95.25 90)
 			(effects
@@
 			)
 		)
-		(property "JLC_Num" "C705627"
+		(property "LCSC" "C705627"
 			(at 119.38 90.17 90)
 			(effects
@@
 			)
 		)
-		(property "JLC_Num" "C464977"
+		(property "LCSC" "C464977"
 			(at 133.35 92.71 0)
 			(effects
@@
 			)
 		)
-		(property "JLC_Num" "C77069"
+		(property "LCSC" "C77069"
 			(at 125.73 99.06 0)
 			(effects

Commit message: feat: m5atom_power_adc 回路・PCB を更新
KiCad 上で行った回路設計・PCB レイアウト変更を反映。
変更内容の詳細は KiCad 上で差分を確認すること。

Co-Authored-By: Claude Sonnet 4.6 <noreply@anthropic.com>
Parts:
- R701: footprint Resistor_SMD:R_0603_1608Metric -> Resistor_SMD:R_0402_1005Metric; LCSC C2989042 -> C2909377
Changed lines of the file:
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@@
 			)
 		)
-		(property "Footprint" "Resistor_SMD:R_0603_1608Metric"
+		(property "Footprint" "Resistor_SMD:R_0402_1005Metric"
 			(at 105.41 90.17 0)
 			(effects
@@
 			)
 		)
-		(property "LCSC" "C2989042"
+		(property "LCSC" "C2909377"
 			(at 105.41 90.17 90)
 			(effects
