File: m5atom_power_adc/power.kicad_sch (KiCad schematic)
At the start: 15 parts, among them Q901 Q_PMOS_GSD, Q902 MMBT2222A, SW901 Boot

Commit message: feat(m5atom_power_adc): リレー状態検出をアナログ分圧からI2C入力に変更
- 分圧抵抗(R201/R202/R301/R302/R401/R402)とRelaySenseラベルを削除
- I2Cコネクタ(J107/J108)を追加、GP2/GP3/GP11/GP12・PWR_HOLDラベルを追加
- +12VAラベルを+12VRAWにリネーム
- ネットクラスの配線幅プリセットに1.0mmを追加
- PCBのネット再割当て・DRC警告を解消

Co-Authored-By: Claude Sonnet 5 <noreply@anthropic.com>
Connections:
- net +12VA renamed +12VRAW
Changed lines of the file:
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@@
 		)
 	)
-	(label "+12VA"
+	(label "+12VRAW"
 		(at 130.81 143.51 0)
 		(effects
@@
 		)
 	)
-	(label "+12VA"
+	(label "+12VRAW"
 		(at 182.88 92.71 180)
 		(effects
