File: m5atom_power_adc/RelayControl.kicad_sch (KiCad schematic)
At the start: 11 parts, among them J201 Relay0, J202 R0SW, Q201 MMBT2222A

Commit message: feat: PCBレイアウト完成・ドキュメントにサブシート構成を反映
- m5atom_power_adc: PCBレイアウト完成（80×82.5mm、131部品、ルーティング完了）
- GroveUnit/RelayControl サブシート更新
- CONTEXT.md/README.md: m5atom_power_adc のファイル構成にサブシート3枚・Library.pretty を追記

Co-Authored-By: Claude Sonnet 4.6 <noreply@anthropic.com>
Parts:
- J201: value Relay0 -> Relay${RIndex}
- J202: value R0SW -> R${RIndex}SW
Connections:
- net GND2 renamed GND1
Changed lines of the file:
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@@
 			)
 		)
-		(property "Value" "Relay0"
+		(property "Value" "Relay${RIndex}"
 			(at 116.84 93.98 0)
 			(effects
@@
 	)
 	(symbol
-		(lib_id "Device:R_Small")
-		(at 118.11 107.95 0)
-		(unit 1)
-		(exclude_from_sim no)
-		(in_bom yes)
-		(on_board yes)
-		(dnp no)
-		(property "Reference" "R201"
-			(at 113.792 107.188 0)
-			(effects
-				(font
-					(size 1.016 1.016)
-				)
-				(justify left)
-			)
-		)
-		(property "Value" "100k"
-			(at 113.03 105.156 0)
-			(effects
-				(font
-					(size 1.27 1.27)
-				)
-				(justify left)
-			)
-		)
-		(property "Footprint" "Resistor_SMD:R_0603_1608Metric"
-			(at 118.11 107.95 0)
-			(effects
-				(font
-					(size 1.27 1.27)
-				)
-				(hide yes)
-			)
-		)
-		(property "Datasheet" "~"
-			(at 118.11 107.95 0)
-			(effects
-				(font
-					(size 1.27 1.27)
-				)
-				(hide yes)
-			)
-		)
-		(property "Description" "Resistor, small symbol"
-			(at 118.11 107.95 0)
-			(effects
-				(font
-					(size 1.27 1.27)
-				)
-				(hide yes)
-			)
-		)
-		(property "JLC_Num" "C2906981"
-			(at 118.11 107.95 0)
-			(effects
-				(font
-					(size 1.27 1.27)
-				)
-				(hide yes)
-			)
-		)
-		(pin "2"
-		)
-		(pin "1"
-		)
-		(instances
-			(project "m5atom_power_adc"
-				(path "/d0098cfc-b338-460c-a156-403456706079/4fe41e33-26ac-47dc-9ee5-c1e37f1f6521"
-					(reference "R201")
-					(unit 1)
-				)
-				(path "/d0098cfc-b338-460c-a156-403456706079/79f1d5f5-7707-41c1-9592-f01b6a759d9e"
-					(reference "R301")
-					(unit 1)
-				)
-				(path "/d0098cfc-b338-460c-a156-403456706079/8c6723eb-7142-4bb9-950b-567c7b549316"
-					(reference "R401")
-					(unit 1)
-				)
-			)
-		)
-	)
-	(symbol
-		(lib_id "power:GND2")
+		(lib_id "power:GND1")
 		(at 121.92 118.11 0)
 		(unit 1)
@@
 			)
 		)
-		(property "Value" "GND2"
+		(property "Value" "GND1"
 			(at 121.92 123.19 0)
 			(effects
@@
 			)
 		)
-		(property "Description" "Power symbol creates a global label with name \"GND2\" , ground"
+		(property "Description" "Power symbol creates a global label with name \"GND1\" , ground"
 			(at 121.92 118.11 0)
 			(effects
@@
 				(path "/d0098cfc-b338-460c-a156-403456706079/8c6723eb-7142-4bb9-950b-567c7b549316"
 					(reference "#PWR0401")
+					(unit 1)
+				)
+			)
+		)
+	)
+	(symbol
+		(lib_id "Device:R_Small")
+		(at 118.11 107.95 0)
+		(unit 1)
+		(exclude_from_sim no)
+		(in_bom yes)
+		(on_board yes)
+		(dnp no)
+		(property "Reference" "R201"
+			(at 113.792 107.188 0)
+			(effects
+				(font
+					(size 1.016 1.016)
+				)
+				(justify left)
+			)
+		)
+		(property "Value" "100k"
+			(at 113.03 105.156 0)
+			(effects
+				(font
+					(size 1.27 1.27)
+				)
+				(justify left)
+			)
+		)
+		(property "Footprint" "Resistor_SMD:R_0603_1608Metric"
+			(at 118.11 107.95 0)
+			(effects
+				(font
+					(size 1.27 1.27)
+				)
+				(hide yes)
+			)
+		)
+		(property "Datasheet" "~"
+			(at 118.11 107.95 0)
+			(effects
+				(font
+					(size 1.27 1.27)
+				)
+				(hide yes)
+			)
+		)
+		(property "Description" "Resistor, small symbol"
+			(at 118.11 107.95 0)
+			(effects
+				(font
+					(size 1.27 1.27)
+				)
+				(hide yes)
+			)
+		)
+		(property "JLC_Num" "C2906981"
+			(at 118.11 107.95 0)
+			(effects
+				(font
+					(size 1.27 1.27)
+				)
+				(hide yes)
+			)
+		)
+		(pin "2"
+		)
+		(pin "1"
+		)
+		(instances
+			(project "m5atom_power_adc"
+				(path "/d0098cfc-b338-460c-a156-403456706079/4fe41e33-26ac-47dc-9ee5-c1e37f1f6521"
+					(reference "R201")
+					(unit 1)
+				)
+				(path "/d0098cfc-b338-460c-a156-403456706079/79f1d5f5-7707-41c1-9592-f01b6a759d9e"
+					(reference "R301")
+					(unit 1)
+				)
+				(path "/d0098cfc-b338-460c-a156-403456706079/8c6723eb-7142-4bb9-950b-567c7b549316"
+					(reference "R401")
 					(unit 1)
 				)
@@
 			)
 		)
-		(property "Value" "R0SW"
+		(property "Value" "R${RIndex}SW"
 			(at 142.24 107.9499 0)
 			(effects

Commit message: chore: PCBネジ穴追加・シルク整理・ロゴ追加・フットプリント修正
- ネジ穴を追加
- シルク文字・ロゴを整理・追加（k_icon フットプリント）
- HY2.0-4PZZ コネクタフットプリントを追加
- 各サブシートのフットプリント修正
- production/ を .gitignore に追加

Co-Authored-By: Claude Sonnet 4.6 <noreply@anthropic.com>
Parts:
- D201: JLC_Num C2128 -> (none); LCSC (none) -> C2128
- D202: JLC_Num C965799 -> (none); LCSC (none) -> C965799
- J201, J202: JLC_Num C158012 -> (none); LCSC (none) -> C158012
- Q201: JLC_Num C8512 -> (none); LCSC (none) -> C8512
- R201: JLC_Num C2906981 -> (none); LCSC (none) -> C2906981
- R202: JLC_Num C22967 -> (none); LCSC (none) -> C22967
- R203, R204, R205: JLC_Num C21190 -> (none); LCSC (none) -> C21190
- TP201: now left out of the parts list
Changed lines of the file:
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@@
 		(unit 1)
 		(exclude_from_sim no)
-		(in_bom yes)
+		(in_bom no)
 		(on_board yes)
 		(dnp no)
@@
 			)
 		)
-		(property "JLC_Num" "C158012"
+		(property "LCSC" "C158012"
 			(at 116.84 100.33 0)
 			(effects
@@
 			)
 		)
-		(property "JLC_Num" "C965799"
+		(property "LCSC" "C965799"
 			(at 133.35 101.6 90)
 			(effects
@@
 			)
 		)
-		(property "JLC_Num" "C21190"
-			(at 129.54 95.25 90)
+		(property "LCSC" "C21190"
+			(at 129.54 95.25 0)
 			(effects
 				(font
@@
 			)
 		)
-		(property "JLC_Num" "C2906981"
+		(property "LCSC" "C2906981"
 			(at 118.11 107.95 0)
 			(effects
@@
 			)
 		)
-		(property "JLC_Num" "C21190"
+		(property "LCSC" "C21190"
 			(at 132.08 113.03 90)
 			(effects
@@
 			)
 		)
-		(property "JLC_Num" "C21190"
-			(at 132.08 95.25 90)
+		(property "LCSC" "C21190"
+			(at 132.08 95.25 0)
 			(effects
 				(font
@@
 			)
 		)
-		(property "JLC_Num" "C158012"
+		(property "LCSC" "C158012"
 			(at 139.7 105.41 0)
 			(effects
@@
 			)
 		)
-		(property "JLC_Num" "C8512"
+		(property "LCSC" "C8512"
 			(at 124.46 113.03 0)
 			(effects
@@
 			)
 		)
-		(property "JLC_Num" "C2128"
+		(property "LCSC" "C2128"
 			(at 125.73 101.6 90)
 			(effects
@@
 			)
 		)
-		(property "JLC_Num" "C22967"
+		(property "LCSC" "C22967"
 			(at 118.11 115.57 0)
 			(effects

Commit message: chore: Grove LED色変更・リレー抵抗を680Ω 500mWに変更・INA228品番更新
Co-Authored-By: Claude Sonnet 4.6 <noreply@anthropic.com>
Parts:
- removed R204: 1k, Resistor_SMD:R_0603_1608Metric, symbol Device:R_Small
- R203: value 1k -> 680 500mW; footprint Resistor_SMD:R_0603_1608Metric -> Resistor_SMD:R_0805_2012Metric; LCSC C21190 -> C543547
Connections:
- net at D202.2 (A): now also R203.2
Changed lines of the file:
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@@
 	(wire
 		(pts
-			(xy 129.54 92.71) (xy 132.08 92.71)
+			(xy 129.54 92.71) (xy 133.35 92.71)
 		)
 		(stroke
@@
 	(wire
 		(pts
-			(xy 132.08 97.79) (xy 133.35 97.79)
-		)
-		(stroke
-			(width 0)
-			(type default)
-		)
-	)
-	(wire
-		(pts
 			(xy 125.73 96.52) (xy 125.73 97.79)
 		)
@@
 		(pts
 			(xy 118.11 118.11) (xy 121.92 118.11)
+		)
+		(stroke
+			(width 0)
+			(type default)
+		)
+	)
+	(wire
+		(pts
+			(xy 133.35 92.71) (xy 133.35 97.79)
 		)
 		(stroke
@@
 			)
 		)
-		(property "Value" "1k"
-			(at 128.524 91.948 0)
-			(effects
-				(font
-					(size 1.27 1.27)
-				)
-			)
-		)
-		(property "Footprint" "Resistor_SMD:R_0603_1608Metric"
+		(property "Value" "680 500mW"
+			(at 132.08 91.694 0)
+			(effects
+				(font
+					(size 1.27 1.27)
+				)
+			)
+		)
+		(property "Footprint" "Resistor_SMD:R_0805_2012Metric"
 			(at 129.54 95.25 0)
 			(effects
@@
 			)
 		)
-		(property "LCSC" "C21190"
+		(property "LCSC" "C543547"
 			(at 129.54 95.25 0)
 			(effects
@@
 					(unit 1)
 				)
-			)
-		)
-	)
-	(symbol
-		(lib_id "Device:R_Small")
-		(at 132.08 95.25 180)
-		(unit 1)
-		(exclude_from_sim no)
-		(in_bom yes)
-		(on_board yes)
-		(dnp no)
-		(property "Reference" "R204"
-			(at 133.096 90.17 0)
-			(effects
-				(font
-					(size 1.016 1.016)
-				)
-			)
-		)
-		(property "Value" "1k"
-			(at 133.096 91.948 0)
-			(effects
-				(font
-					(size 1.27 1.27)
-				)
-			)
-		)
-		(property "Footprint" "Resistor_SMD:R_0603_1608Metric"
-			(at 132.08 95.25 0)
-			(effects
-				(font
-					(size 1.27 1.27)
-				)
-				(hide yes)
-			)
-		)
-		(property "Datasheet" "~"
-			(at 132.08 95.25 0)
-			(effects
-				(font
-					(size 1.27 1.27)
-				)
-				(hide yes)
-			)
-		)
-		(property "Description" "Resistor, small symbol"
-			(at 132.08 95.25 0)
-			(effects
-				(font
-					(size 1.27 1.27)
-				)
-				(hide yes)
-			)
-		)
-		(property "LCSC" "C21190"
-			(at 132.08 95.25 0)
-			(effects
-				(font
-					(size 1.27 1.27)
-				)
-				(hide yes)
-			)
-		)
-		(pin "2"
-		)
-		(pin "1"
-		)
-		(instances
-			(project "m5atom_power_adc"
-				(path "/d0098cfc-b338-460c-a156-403456706079/4fe41e33-26ac-47dc-9ee5-c1e37f1f6521"
-					(reference "R204")
-					(unit 1)
-				)
-				(path "/d0098cfc-b338-460c-a156-403456706079/79f1d5f5-7707-41c1-9592-f01b6a759d9e"
-					(reference "R304")
-					(unit 1)
-				)
-				(path "/d0098cfc-b338-460c-a156-403456706079/8c6723eb-7142-4bb9-950b-567c7b549316"
-					(reference "R404")
-					(unit 1)
-				)

Commit message: feat: m5atom_power_adc 回路・PCB を更新
KiCad 上で行った回路設計・PCB レイアウト変更を反映。
変更内容の詳細は KiCad 上で差分を確認すること。

Co-Authored-By: Claude Sonnet 4.6 <noreply@anthropic.com>
Parts:
- R201: LCSC C2906981 -> C25803
- R203: value 680 500mW -> 1.5k; footprint Resistor_SMD:R_0805_2012Metric -> Resistor_SMD:R_1206_3216Metric; LCSC C543547 -> C114929
Changed lines of the file:
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@@
 			)
 		)
-		(property "Value" "680 500mW"
+		(property "Value" "1.5k"
 			(at 132.08 91.694 0)
 			(effects
@@
 			)
 		)
-		(property "Footprint" "Resistor_SMD:R_0805_2012Metric"
+		(property "Footprint" "Resistor_SMD:R_1206_3216Metric"
 			(at 129.54 95.25 0)
 			(effects
@@
 			)
 		)
-		(property "LCSC" "C543547"
+		(property "LCSC" "C114929"
 			(at 129.54 95.25 0)
 			(effects
@@
 			)
 		)
-		(property "LCSC" "C2906981"
-			(at 118.11 107.95 0)
-			(effects
+		(property "LCSC" "C25803"
+			(at 118.11 107.95 0)
+			(effects

Commit message: feat(m5atom_power_adc): 逆極性保護を理想ダイオード(LM73100)に置き換え、電源スイッチ＆自己保持回路を追加（作業途中）
- LM73100用カスタム記号・フットプリント(VQFN-10-HR)を追加
- 電源回路をサブシートに分離(power.kicad_sch)
- PCBレイアウト更新

Co-Authored-By: Claude Sonnet 4.6 <noreply@anthropic.com>
Parts:
- renumbered R205 to R204
Changed lines of the file:
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@@
 		(on_board yes)
 		(dnp no)
-		(property "Reference" "R205"
+		(property "Reference" "R204"
 			(at 134.366 109.474 90)
 			(effects
@@
 			(project "m5atom_power_adc"
 				(path "/d0098cfc-b338-460c-a156-403456706079/4fe41e33-26ac-47dc-9ee5-c1e37f1f6521"
-					(reference "R205")
+					(reference "R204")
 					(unit 1)
 				)
 				(path "/d0098cfc-b338-460c-a156-403456706079/79f1d5f5-7707-41c1-9592-f01b6a759d9e"
-					(reference "R305")
+					(reference "R304")
 					(unit 1)
 				)
 				(path "/d0098cfc-b338-460c-a156-403456706079/8c6723eb-7142-4bb9-950b-567c7b549316"
-					(reference "R405")
+					(reference "R404")
 					(unit 1)
 				)

Commit message: feat(m5atom_power_adc): リレー状態検出をアナログ分圧からI2C入力に変更
- 分圧抵抗(R201/R202/R301/R302/R401/R402)とRelaySenseラベルを削除
- I2Cコネクタ(J107/J108)を追加、GP2/GP3/GP11/GP12・PWR_HOLDラベルを追加
- +12VAラベルを+12VRAWにリネーム
- ネットクラスの配線幅プリセットに1.0mmを追加
- PCBのネット再割当て・DRC警告を解消

Co-Authored-By: Claude Sonnet 5 <noreply@anthropic.com>
Parts:
- removed R201: 100k, Resistor_SMD:R_0603_1608Metric, symbol Device:R_Small
- removed R202: 27k, Resistor_SMD:R_0603_1608Metric, symbol Device:R_Small
Changed lines of the file:
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@@
-	)
-	(junction
-		(at 118.11 111.76)
-		(diameter 0)
-		(color 0 0 0 0)
 	)
 	(junction
@@
 	(wire
 		(pts
-			(xy 111.76 111.76) (xy 118.11 111.76)
-		)
-		(stroke
-			(width 0)
-			(type default)
-		)
-	)
-	(wire
-		(pts
 			(xy 121.92 105.41) (xy 125.73 105.41)
 		)
@@
 	(wire
 		(pts
-			(xy 118.11 118.11) (xy 121.92 118.11)
-		)
-		(stroke
-			(width 0)
-			(type default)
-		)
-	)
-	(wire
-		(pts
 			(xy 133.35 92.71) (xy 133.35 97.79)
 		)
@@
 	(wire
 		(pts
-			(xy 118.11 110.49) (xy 118.11 111.76)
-		)
-		(stroke
-			(width 0)
-			(type default)
-		)
-	)
-	(wire
-		(pts
 			(xy 129.54 97.79) (xy 125.73 97.79)
 		)
@@
 		(pts
 			(xy 121.92 97.79) (xy 125.73 97.79)
-		)
-		(stroke
-			(width 0)
-			(type default)
-		)
-	)
-	(wire
-		(pts
-			(xy 118.11 105.41) (xy 121.92 105.41)
-		)
-		(stroke
-			(width 0)
-			(type default)
-		)
-	)
-	(wire
-		(pts
-			(xy 118.11 111.76) (xy 118.11 113.03)
 		)
 		(stroke
@@
 		(shape input)
 		(at 137.16 113.03 0)
-		(effects
-			(font
-				(size 1.27 1.27)
-			)
-			(justify left)
-		)
-	)
-	(hierarchical_label "RelaySense"
-		(shape output)
-		(at 111.76 111.76 90)
 		(effects
 			(font
@@
 	(symbol
 		(lib_id "Device:R_Small")
-		(at 118.11 107.95 0)
-		(unit 1)
-		(exclude_from_sim no)
-		(in_bom yes)
-		(on_board yes)
-		(dnp no)
-		(property "Reference" "R201"
-			(at 113.792 107.188 0)
-			(effects
-				(font
-					(size 1.016 1.016)
-				)
-				(justify left)
-			)
-		)
-		(property "Value" "100k"
-			(at 113.03 105.156 0)
-			(effects
-				(font
-					(size 1.27 1.27)
-				)
-				(justify left)
-			)
-		)
-		(property "Footprint" "Resistor_SMD:R_0603_1608Metric"
-			(at 118.11 107.95 0)
-			(effects
-				(font
-					(size 1.27 1.27)
-				)
-				(hide yes)
-			)
-		)
-		(property "Datasheet" "~"
-			(at 118.11 107.95 0)
-			(effects
-				(font
-					(size 1.27 1.27)
-				)
-				(hide yes)
-			)
-		)
-		(property "Description" "Resistor, small symbol"
-			(at 118.11 107.95 0)
-			(effects
-				(font
-					(size 1.27 1.27)
-				)
-				(hide yes)
-			)
-		)
-		(property "LCSC" "C25803"
-			(at 118.11 107.95 0)
-			(effects
-				(font
-					(size 1.27 1.27)
-				)
-				(hide yes)
-			)
-		)
-		(pin "2"
-		)
-		(pin "1"
-		)
-		(instances
-			(project "m5atom_power_adc"
-				(path "/d0098cfc-b338-460c-a156-403456706079/4fe41e33-26ac-47dc-9ee5-c1e37f1f6521"
-					(reference "R201")
-					(unit 1)
-				)
-				(path "/d0098cfc-b338-460c-a156-403456706079/79f1d5f5-7707-41c1-9592-f01b6a759d9e"
-					(reference "R301")
-					(unit 1)
-				)
-				(path "/d0098cfc-b338-460c-a156-403456706079/8c6723eb-7142-4bb9-950b-567c7b549316"
-					(reference "R401")
-					(unit 1)
-				)
-			)
-		)
-	)
-	(symbol
-		(lib_id "Device:R_Small")
 		(at 132.08 113.03 90)
 		(unit 1)
@@
 					(unit 1)
 				)
-			)
-		)
-	)
-	(symbol
-		(lib_id "Device:R_Small")
-		(at 118.11 115.57 0)
-		(unit 1)
-		(exclude_from_sim no)
-		(in_bom yes)
-		(on_board yes)
-		(dnp no)
-		(property "Reference" "R202"
-			(at 114.046 114.554 0)
-			(effects
-				(font
-					(size 1.016 1.016)
-				)
-				(justify left)
-			)
-		)
-		(property "Value" "27k"
-			(at 113.03 116.586 0)
-			(effects
-				(font
-					(size 1.27 1.27)
-				)
-				(justify left)
-			)
-		)
-		(property "Footprint" "Resistor_SMD:R_0603_1608Metric"
-			(at 118.11 115.57 0)
-			(effects
-				(font
-					(size 1.27 1.27)
-				)
-				(hide yes)
-			)
-		)
-		(property "Datasheet" "~"
-			(at 118.11 115.57 0)
-			(effects
-				(font
-					(size 1.27 1.27)
-				)
-				(hide yes)
-			)
-		)
-		(property "Description" "Resistor, small symbol"
-			(at 118.11 115.57 0)
-			(effects
-				(font
-					(size 1.27 1.27)
-				)
-				(hide yes)
-			)
-		)
-		(property "LCSC" "C22967"
-			(at 118.11 115.57 0)
-			(effects
-				(font
-					(size 1.27 1.27)
-				)
-				(hide yes)
-			)
-		)
-		(pin "2"
-		)
-		(pin "1"
-		)
-		(instances
-			(project "m5atom_power_adc"
-				(path "/d0098cfc-b338-460c-a156-403456706079/4fe41e33-26ac-47dc-9ee5-c1e37f1f6521"
-					(reference "R202")
-					(unit 1)
-				)
-				(path "/d0098cfc-b338-460c-a156-403456706079/79f1d5f5-7707-41c1-9592-f01b6a759d9e"
-					(reference "R302")
-					(unit 1)
-				)
-				(path "/d0098cfc-b338-460c-a156-403456706079/8c6723eb-7142-4bb9-950b-567c7b549316"
-					(reference "R402")
-					(unit 1)
-				)

Commit message: feat: ACC検知回路（IGN連動deep sleep復帰用）を追加
分圧を使わず、車のACC(12V)をD109(BZT52C15ツェナー保護)→Q105(PDTC114YU,115デジタルトランジスタ)→R111(10kΩプルアップ)経由でGPIO1に直接入力する回路を追加。ACC ONでGPIO1がLOWになり、ext1 wakeup(ANY_LOW)でdeep sleepから復帰させる想定。

- GPIO1はstrapping pinに該当せずRTC GPIO対応のため採用
- コネクタ用スペースがなくスルーホールパッド1点で対応、GND側はNetTieで共通化済みのGND1を流用し省略
- Q105のEmitterは配線都合でGND2ではなくGND1に接続
- ファームウェア未実装。電源保持・理想ダイオード回路の検証用テストボード製造・テストを先に行う方針

Co-Authored-By: Claude Sonnet 5 <noreply@anthropic.com>
Other:
- moved on the sheet: J201, J202
Changed lines of the file:
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@@
+	)
+	(junction
+		(at 121.92 105.41)
+		(diameter 0)
+		(color 0 0 0 0)
 	)
 	(junction
@@
 	)
 	(junction
-		(at 121.92 105.41)
-		(diameter 0)
-		(color 0 0 0 0)
-	)
-	(junction
-		(at 133.35 105.41)
+		(at 118.11 105.41)
 		(diameter 0)
 		(color 0 0 0 0)
@@
 	(wire
 		(pts
-			(xy 128.27 107.95) (xy 128.27 118.11)
+			(xy 118.11 114.3) (xy 118.11 118.11)
+		)
+		(stroke
+			(width 0)
+			(type default)
+		)
+	)
+	(wire
+		(pts
+			(xy 118.11 105.41) (xy 121.92 105.41)
 		)
 		(stroke
@@
 	(wire
 		(pts
+			(xy 133.35 92.71) (xy 133.35 97.79)
+		)
+		(stroke
+			(width 0)
+			(type default)
+		)
+	)
+	(wire
+		(pts
+			(xy 118.11 118.11) (xy 121.92 118.11)
+		)
+		(stroke
+			(width 0)
+			(type default)
+		)
+	)
+	(wire
+		(pts
+			(xy 129.54 97.79) (xy 125.73 97.79)
+		)
+		(stroke
+			(width 0)
+			(type default)
+		)
+	)
+	(wire
+		(pts
+			(xy 118.11 100.33) (xy 118.11 105.41)
+		)
+		(stroke
+			(width 0)
+			(type default)
+		)
+	)
+	(wire
+		(pts
+			(xy 121.92 105.41) (xy 121.92 107.95)
+		)
+		(stroke
+			(width 0)
+			(type default)
+		)
+	)
+	(wire
+		(pts
+			(xy 118.11 97.79) (xy 125.73 97.79)
+		)
+		(stroke
+			(width 0)
+			(type default)
+		)
+	)
+	(wire
+		(pts
+			(xy 118.11 105.41) (xy 118.11 111.76)
+		)
+		(stroke
+			(width 0)
+			(type default)
+		)
+	)
+	(wire
+		(pts
 			(xy 121.92 105.41) (xy 125.73 105.41)
-		)
-		(stroke
-			(width 0)
-			(type default)
-		)
-	)
-	(wire
-		(pts
-			(xy 128.27 118.11) (xy 121.92 118.11)
-		)
-		(stroke
-			(width 0)
-			(type default)
-		)
-	)
-	(wire
-		(pts
-			(xy 133.35 92.71) (xy 133.35 97.79)
-		)
-		(stroke
-			(width 0)
-			(type default)
-		)
-	)
-	(wire
-		(pts
-			(xy 129.54 97.79) (xy 125.73 97.79)
-		)
-		(stroke
-			(width 0)
-			(type default)
-		)
-	)
-	(wire
-		(pts
-			(xy 121.92 100.33) (xy 121.92 105.41)
-		)
-		(stroke
-			(width 0)
-			(type default)
-		)
-	)
-	(wire
-		(pts
-			(xy 121.92 97.79) (xy 125.73 97.79)
-		)
-		(stroke
-			(width 0)
-			(type default)
-		)
-	)
-	(wire
-		(pts
-			(xy 133.35 105.41) (xy 134.62 105.41)
-		)
-		(stroke
-			(width 0)
-			(type default)
-		)
-	)
-	(wire
-		(pts
-			(xy 121.92 105.41) (xy 121.92 107.95)
-		)
-		(stroke
-			(width 0)
-			(type default)
-		)
-	)
-	(wire
-		(pts
-			(xy 134.62 107.95) (xy 128.27 107.95)
 		)
 		(stroke
@@
 	(symbol
 		(lib_id "Connector_Generic:Conn_01x02")
-		(at 116.84 100.33 180)
+		(at 113.03 100.33 180)
 		(unit 1)
 		(exclude_from_sim no)
@@
 		(dnp no)
 		(property "Reference" "J201"
-			(at 116.84 91.44 0)
+			(at 113.03 91.44 0)
 			(effects
 				(font
@@
 		)
 		(property "Value" "Relay${RIndex}"
-			(at 116.84 93.98 0)
+			(at 113.03 93.98 0)
 			(effects
 				(font
@@
 		)
 		(property "Footprint" "Connector_JST:JST_XH_B2B-XH-A_1x02_P2.50mm_Vertical"
-			(at 116.84 100.33 0)
+			(at 113.03 100.33 0)
 			(effects
 				(font
@@
 		)
 		(property "Datasheet" "~"
-			(at 116.84 100.33 0)
+			(at 113.03 100.33 0)
 			(effects
 				(font
@@
 		)
 		(property "Description" "Generic connector, single row, 01x02, script generated (kicad-library-utils/schlib/autogen/connector/)"
-			(at 116.84 100.33 0)
+			(at 113.03 100.33 0)
 			(effects
 				(font
@@
 		)
 		(property "LCSC" "C158012"
-			(at 116.84 100.33 0)
+			(at 113.03 100.33 0)
 			(effects
 				(font
@@
 	(symbol
 		(lib_id "Connector_Generic:Conn_01x02")
-		(at 139.7 105.41 0)
+		(at 113.03 111.76 0)
+		(mirror y)
 		(unit 1)
 		(exclude_from_sim no)
@@
 		(dnp no)
 		(property "Reference" "J202"
-			(at 142.24 105.4099 0)
+			(at 110.49 111.7599 0)
 			(effects
 				(font
@@
 		)
 		(property "Value" "R${RIndex}SW"
-			(at 142.24 107.9499 0)
+			(at 110.49 114.2999 0)
 			(effects
 				(font
@@
 		)
 		(property "Footprint" "Connector_JST:JST_XH_B2B-XH-A_1x02_P2.50mm_Vertical"
-			(at 139.7 105.41 0)
+			(at 113.03 111.76 0)
 			(effects
 				(font
@@
 		)
 		(property "Datasheet" "~"
-			(at 139.7 105.41 0)
+			(at 113.03 111.76 0)
 			(effects
 				(font
@@
 		)
 		(property "Description" "Generic connector, single row, 01x02, script generated (kicad-library-utils/schlib/autogen/connector/)"
-			(at 139.7 105.41 0)
+			(at 113.03 111.76 0)
 			(effects
 				(font
@@
 		)
 		(property "LCSC" "C158012"
-			(at 139.7 105.41 0)
-			(effects
-				(font
+			(at 113.03 111.76 0)
+			(effects
+				(font
